File: 4_Wave_Generador/4_Wave_Generator.sch (KiCad schematic (older format))
At the start: 102 parts, among them J1 RS232, J10 Jumper, J11 Jumper, J12 Jumper, J13 Jumper, J14 Jumper, J15 Jumper, J2 I2C, J3 SPEAKER, J4 RESET, J7 Jumper, J8 Jumper, J9 Jumper, P1 ECG INPUTS, P2 PIC_PROGRAMER, P3 SPI, P4 AD8232_CONTROL, P5 PIC_OUTPUTS, P6 CONN_01X04, P7 CONN_01X04, P8 MCLK_EXTERNAL, SW1 SW_Push, SW2 RESET_PIC, U1 AD8232_A, U2 PIC16F688, U3 AD8421, U4 AD9833, U5 ADG819, U6 LD1117S33TR_MIO, U7 ATMEGA328P-AU_MIO, Y1 Crystal_8MHz, Y2 Crystal

Commit message: GENERADOR_V1
ARREGLO ESQUEMATICO
Parts:
- removed U2: PIC16F688, Housings_SOIC:SOIC-14_3.9x8.7mm_Pitch1.27mm, symbol PIC16F688
- added J?: Jumper, Pin_Headers:Pin_Header_Straight_1x02_Pitch2.54mm, symbol Jumper-RESCUE-PCB_OSCILLATOR
- added J?: RS232_PIC, Foot_Prints_Manager_Outputs:RS232, symbol CONN_01X03
- added P?: SALIDAS_DIG_ATMEGA, symbol CONN_01X11
- added P?: SALIDAS_DIG_PIC, symbol CONN_01X05
- added P?: ENTRADA_OXIMETRO, symbol CONN_02X03
- added U?: PIC16F688, Housings_SOIC:SOIC-14_3.9x8.7mm_Pitch1.27mm, symbol PIC16F688
Connections:
- net labels added: OSC1, OSC2, OXI_1, OXI_2, OXI_3, PB0, PB1, PC0, PC1, PC2, PC3, PD2, PD3, PD4, PD5, PD6, PD7, RC0_PIC, RC1_PIC, RC2_PIC, RC3_PIC, RX_PIC, TX_PIC
- wire segments 297 -> 330
Other:
- note added: "MICROCONTROLADOR \nATMEGA 328P"
- note added: "PIC16F688"
- note removed: "CONVERTIDOR ANALOGICO A DIGITAL\n"
- moved on the sheet: C10, C13, C15, C18, C19, C25, C26, C27, C31, C32, C33, D3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

Commit message: GENERADOR_V2
TEST POIN
Parts:
- removed J?: Jumper, Pin_Headers:Pin_Header_Straight_1x02_Pitch2.54mm, symbol Jumper-RESCUE-PCB_OSCILLATOR
- removed P5: PIC_OUTPUTS, Pin_Headers:Pin_Header_Straight_1x03_Pitch2.54mm, symbol CONN_01X03
- removed U1: AD8232_A, Huellas:AD8232_ECG, symbol AD8232_A
- removed U?: PIC16F688, Housings_SOIC:SOIC-14_3.9x8.7mm_Pitch1.27mm, symbol PIC16F688
- added JP?: AREF, Pin_Headers:Pin_Header_Straight_1x02_Pitch2.54mm, symbol PASO_A/D
- added U?: PIC16F688, Housings_SOIC:SOIC-14_3.9x8.7mm_Pitch1.27mm, symbol PIC16F688
- added U?: AD8232_A, Huellas:AD8232_ECG, symbol AD8232_A
- added W? (x4): TEST_1P, symbol TEST_1P
Connections:
- net +vs: now also U?.17 (+VS)
- net GND: now also C13.2, U?.14 (AC/DC), U?.14 (VSS), U?.16 (GND)
- net IAOUT: now also U?.19 (IAOUT)
- net ICSPCLK: now also U?.12 (ICSPCLK)
- net ICSPDAT: now also U?.13 (ICSPDAT)
- net LOD+: now also U?.12 (LOD+)
- net LOD-: now also U?.11 (LOD-)
- net MCLR/Vpp: now also U?.4 (MCLR/Vpp)
- net OPAMP+: now also U?.7 (OPAMP+)
- net OSC1: now also U?.2 (OSC1)
- net OSC2: now also U?.3 (OSC2)
- net OUT_ANALOG: now also U?.10 (OUT), W?.1
- net RC1_PIC: now also U?.9 (RC1)
- net RC2_PIC: now also U?.8 (RC2)
- net RC3_PIC: now also U?.7 (RC3)
- net REFIN: now also U?.18 (REFIN)
- net REFOUT: now also U?.8 (REFOUT)
- net RLD: now also U?.5 (RLD)
- net RLDFB: now also U?.4 (RLDFB)
- net RX_PIC: now also U?.5 (RX)
- net SDN: now also U?.13 (SDN)
- net SW: now also U?.6 (SW)
- net TX_PIC: now also U?.6 (TX)
- net VDD: now also C13.1, JP?.1, U?.1 (VDD), U?.15 (FR)
- net at U7.20 (AREF): now also JP?.2
- net at R5.2: now also U?.2 (+IN)
- net at R6.2: now also U?.3 (-IN)
- net at R13.2, R15.1: now also U?.9 (OPAMP-)
- net at C3.1, R8.2: now also U?.20 (HPSENSE)
- net at C3.2: now also U?.1 (HPDRIVE)
- net ADC renamed ADC_1
- net ADC_1: now also U?.11 (RA2), W?.1
- new net ADC_2: U?.10 (RC0), W?.1
Other:
- note added: "SALIDAS DE DIGITALES"
- note removed: "ACTUALIZAR CON TODAS LAS SALIDAS"
- moved on the sheet: C11, C12, C13, C14, C15, C16, C17, C8, C9, P4

Commit message: GENERADOR_V3
VISTO
Parts:
- removed J3: SPEAKER, Pin_Headers:Pin_Header_Angled_1x02_Pitch2.54mm, symbol CONN_01X02
- removed U7: ATMEGA328P-AU_MIO, Housings_QFP:TQFP-32_7x7mm_Pitch0.8mm, symbol ATMEGA328P-AU_MIO
- added U?: ATMEGA328P-AU_MIO, Housings_QFP:TQFP-32_7x7mm_Pitch0.8mm, symbol ATMEGA328P-AU_MIO
- added W? (x8): TEST_1P, symbol TEST_1P
Connections:
- net +12V: now also W?.1
- net -12V: now also W?.1
- net BASE_WAVE: now also W?.1
- net GND: now also U?.21 (GND), U?.3 (GND), U?.5 (GND), W?.1
- net MCLK_DDS_1: now also W?.1
- net MISO: now also U?.16 ((PCINT4/MISO)PB4)
- net MOSI: now also U?.15 ((PCINT3/OC2A/MOSI)PB3)
- net PB0: now also U?.12 ((PCINT0/CLKO/ICP1)PB0)
- net PB1: now also U?.13 ((PCINT1/OC1A)PB1)
- net PC0: now also U?.23 ((PCINT8/ADC0)PC0)
- net PC1: now also U?.24 ((PCINT9/ADC1)PC1)
- net PC2: now also U?.25 ((PCINT10/ADC2)PC2)
- net PC3: now also U?.26 ((PCINT11/ADC3)PC3)
- net PD2: now also U?.32 ((PCINT18/INT0)PD2)
- net PD3: now also U?.1 ((PCINT19/OC2B/INT1)PD3)
- net PD4: now also U?.2 ((PCINT20/XCK/T0)PD4)
- net PD5: now also U?.9 ((PCINT21/OC0B/T1)PD5)
- net PD6: now also U?.10 ((PCINT22/OC0A/AIN0)PD6)
- net PD7: now also U?.11 ((PCINT23/AIN1)PD7)
- net RESET: now also U?.29 ((PCINT14/~RESET~)PC6)
- net Rx: now also U?.30 ((PCINT16/RXD)PD0)
- net SCK: now also U?.17 ((PCINT5/SCK)PB5)
- net SCL: now also U?.28 ((PCINT13/SCL/ADC5)PC5)
- net SDA: now also U?.27 ((PCINT12/SDA/ADC4)PC4)
- net SS: now also U?.14 ((PCINT2/OC1B/~SS~)PB2)
- net Tx: now also U?.31 ((PCINT17/TXD)PD1)
- net VDD: now also U?.18 (AVCC), U?.4 (VCC), U?.6 (VCC), W?.1
- net WAVE_DDS_1: now also W?.1
- net XTAL1: now also U?.7 ((PCINT6/XTAL1/TOSC1)PB6)
- net XTAL2: now also U?.8 ((PCINT7/XTAL2/TOSC2)PB7)
- net at JP?.2: now also U?.20 (AREF)
- net MODULATED_WAVE renamed MODULATED_WAVE_1
- net MODULATED_WAVE_1: now also W?.1; no longer J?.1
- new net MODULATED_WAVE_2: J?.1, W?.1
Other:
- note added: "INPUT ECG // OXIMETRO\n"
- note added: "OUTPUT OF DIGITAL"
- note added: "TEST POINTS\n"
- note removed: "SALIDAS DE DIGITALES"
- moved on the sheet: D3, D5, D7, D?, J2, J4, P4, P6, P7, R2, R22, R23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

Commit message: GENERADOR_V4
CAMBIO DE DATASHEEP Y ARREGLO DE SEÑALES
Parts:
- removed CLK1: KC5032A, Foot_Prints_PCB_OSCILLATOR:KC5032A_Foot_Print, symbol KC5032A
- removed J8, J9: Jumper, Pin_Headers:Pin_Header_Straight_1x02_Pitch2.54mm, symbol Jumper-RESCUE-PCB_OSCILLATOR
- removed U3: AD8421, Housings_SOIC:SOIC-8_3.9x4.9mm_Pitch1.27mm, symbol AD8421
- removed U5, U?: ADG819, Housings_SSOP:MSOP-8_3x3mm_Pitch0.65mm, symbol ADG819
- added CLK?: KC5032A, Foot_Prints_PCB_OSCILLATOR:KC5032A_Foot_Print, symbol KC5032A
- added P?: RG_8421, symbol CONN_01X02
- added U? (x2): ADG819, Housings_SSOP:MSOP-8_3x3mm_Pitch0.65mm, symbol ADG819
- added U?: AD8421, symbol AD8421
Connections:
- net +12V: now also U?.8 (+Vs)
- net -12V: now also U?.5 (-Vs)
- net A_AD5270_1: now also P?.1 (P1), U?.2 (Rg)
- net BASE_WAVE: now also U?.8 (S2), U?.8 (S2)
- net GND: now also CLK?.2 (GND), U?.1 (-IN), U?.2 (S1), U?.2 (S1), U?.3 (GND), U?.3 (GND)
- net MCLK_DDS_1: now also CLK?.3 (Output)
- net MODULATING_WAVE: now also U?.6 (IN), U?.6 (IN)
- net VDD: now also CLK?.4 (Vcc), U?.4 (VDD), U?.4 (VDD)
- net W_AD5270_1: now also P?.2 (P2), U?.3 (Rg)
- net at J12.1: now also U?.6 (REF)
- net at J13.2: now also U?.7 (Vout)
- net at J7.1, R21.2: now also CLK?.1 (_INH)
- net at J15.2: now also U?.1 (D)
- net at J?.2: now also U?.1 (D)
- new net WAVE_DDS_2: U?.4 (+IN)
Changed lines of the file:
@@
 Text Notes 10980 4790 0    60   ~ 0
 CLOK_DDS_1
-$Comp
-L AD8421 U3
-U 1 1 59D306B2
-P 14530 3400
-F 0 "U3" H 14310 3710 60  0000 C CNN
-F 1 "AD8421" H 14520 3330 60  0000 C CNN
-F 2 "Housings_SOIC:SOIC-8_3.9x4.9mm_Pitch1.27mm" H 14360 3100 60  0001 C CNN
-F 3 "" H 14360 3100 60  0000 C CNN
-	1    14530 3400
-	1    0    0    -1
-$EndComp
 Text Label 14570 2700 3    60   ~ 0
 +12V
@@
 WAVE_DDS_1
 Text Label 13410 3210 0    60   ~ 0
-WAVE_DDS_1
+WAVE_DDS_2
 Text Label 13830 3810 1    60   ~ 0
 GND
@@
 	-1   0    0    1
 $EndComp
-$Comp
-L KC5032A CLK1
-U 1 1 59D306C4
-P 11220 5060
-F 0 "CLK1" H 11220 5260 60  0000 C CNN
-F 1 "KC5032A" H 11220 5060 60  0000 C CNN
-F 2 "Foot_Prints_PCB_OSCILLATOR:KC5032A_Foot_Print" H 11160 5070 60  0001 C CNN
-F 3 "" H 11160 5070 60  0000 C CNN
-F 4 "1253-1043-2-ND" H 11320 5360 60  0001 C CNN "OSC XO 25.000MHZ CMOS SMD"
-	1    11220 5060
-	1    0    0    -1
-$EndComp
 NoConn ~ 14790 5730
 NoConn ~ 14790 5840
@@
 Text Label 15260 1060 0    60   ~ 0
 VDD
-$Comp
-L Jumper-RESCUE-PCB_OSCILLATOR J8
-U 1 1 59D306C7
-P 13810 3360
-F 0 "J8" V 13770 3420 50  0000 L CNN
-F 1 "Jumper" H 13840 3320 50  0001 L CNN
-F 2 "Pin_Headers:Pin_Header_Straight_1x02_Pitch2.54mm" H 13740 3280 50  0001 C CNN
-F 3 "" H 13810 3360 50  0000 C CNN
-	1    13810 3360
-	0    1    1    0
-$EndComp
-$Comp
-L Jumper-RESCUE-PCB_OSCILLATOR J9
-U 1 1 59D306C8
-P 13810 3460
-F 0 "J9" V 13780 3530 50  0000 L CNN
-F 1 "Jumper" H 13840 3420 50  0001 L CNN
-F 2 "Pin_Headers:Pin_Header_Straight_1x02_Pitch2.54mm" H 13740 3380 50  0001 C CNN
-F 3 "" H 13810 3460 50  0000 C CNN
-	1    13810 3460
-	0    1    1    0
-$EndComp
 $Comp
 L Jumper-RESCUE-PCB_OSCILLATOR J13
@@
 	13830 3620 13830 3810
 Wire Wire Line
-	13910 3360 13970 3360
-Wire Wire Line
-	13970 3460 13910 3460
-Wire Wire Line
-	13160 3360 13710 3360
-Wire Wire Line
-	13160 3460 13710 3460
+	13160 3360 13970 3360
+Wire Wire Line
+	13160 3460 13970 3460
 Wire Wire Line
 	14880 2910 14880 2870
@@
 Wire Wire Line
 	14790 3930 14790 3980
-$Comp
-L ADG819 U5
-U 1 1 59D306CF
-P 14390 5800
-F 0 "U5" H 14250 6180 60  0000 C CNN
-F 1 "ADG819" H 14400 5800 60  0000 C CNN
-F 2 "Housings_SSOP:MSOP-8_3x3mm_Pitch0.65mm" H 14150 6080 60  0001 C CNN
-F 3 "" H 14390 5800 60  0000 C CNN
-	1    14390 5800
-	1    0    0    -1
-$EndComp
 $Comp
 L 10K R21
@@
 Wire Wire Line
 	15260 7810 15260 8760
-$Comp
-L ADG819 U?
-U 1 1 59DE4715
-P 14370 8010
-F 0 "U?" H 14230 8390 60  0000 C CNN
-F 1 "ADG819" H 14380 8010 60  0000 C CNN
-F 2 "Housings_SSOP:MSOP-8_3x3mm_Pitch0.65mm" H 14130 8290 60  0001 C CNN
-F 3 "" H 14370 8010 60  0000 C CNN
-	1    14370 8010
-	1    0    0    -1
-$EndComp
 Text Label 13270 7920 0    60   ~ 0
 BASE_WAVE
@@
 Text Label 7950 9240 1    60   ~ 0
 MODULATED_WAVE_2
+$Comp
+L CONN_01X02 P?
+U 1 1 59D428FA
+P 10370 8100
+F 0 "P?" H 10370 8250 50  0000 C CNN
+F 1 "RG_8421" V 10470 8100 50  0000 C CNN
+F 2 "" H 10370 8100 50  0000 C CNN
+F 3 "" H 10370 8100 50  0000 C CNN
+	1    10370 8100
+	0    -1   -1   0
+$EndComp
+Wire Wire Line
+	10320 8300 10320 9070
+Wire Wire Line
+	10420 8300 10420 9070
+Text Label 10320 9070 1    60   ~ 0
+A_AD5270_1
+Text Label 10420 9070 1    60   ~ 0
+W_AD5270_1
+$Comp
+L ADG819 U?
+U 1 1 59D73BBE
+P 14370 8010
+F 0 "U?" H 14230 8390 60  0000 C CNN
+F 1 "ADG819" H 14380 8010 60  0000 C CNN
+F 2 "Housings_SSOP:MSOP-8_3x3mm_Pitch0.65mm" H 14130 8290 60  0001 C CNN
+F 3 "" H 14370 8010 60  0000 C CNN
+	1    14370 8010
+	1    0    0    -1
+$EndComp
+$Comp
+L ADG819 U?
+U 1 1 59D744EC
+P 14390 5800
+F 0 "U?" H 14250 6180 60  0000 C CNN
+F 1 "ADG819" H 14400 5800 60  0000 C CNN
+F 2 "Housings_SSOP:MSOP-8_3x3mm_Pitch0.65mm" H 14150 6080 60  0001 C CNN
+F 3 "" H 14390 5800 60  0000 C CNN
+	1    14390 5800
+	1    0    0    -1
+$EndComp
+$Comp
+L AD8421 U?
+U 1 1 59D78D88
+P 14530 3400
+F 0 "U?" H 14310 3710 60  0000 C CNN
+F 1 "AD8421" H 14520 3330 60  0000 C CNN
+F 2 "" H 14360 3100 60  0000 C CNN
+F 3 "" H 14360 3100 60  0000 C CNN
+	1    14530 3400
+	1    0    0    -1
+$EndComp
+$Comp
+L KC5032A CLK?
+U 1 1 59D7E65A
+P 11220 5060
+F 0 "CLK?" H 11220 5260 60  0000 C CNN
+F 1 "KC5032A" H 11220 5060 60  0000 C CNN
+F 2 "Foot_Prints_PCB_OSCILLATOR:KC5032A_Foot_Print" H 11160 5070 60  0001 C CNN
+F 3 "" H 11160 5070 60  0000 C CNN
+F 4 "1253-1043-2-ND" H 11320 5360 60  0001 C CNN "OSC XO 25.000MHZ CMOS SMD"
+	1    11220 5060
+	1    0    0    -1
+$EndComp
 $EndSCHEMATC

Commit message: GENERADOR V5
POR FIN HUELLAS Y DATASHEEP
Parts:
- removed CLK?: KC5032A, Foot_Prints_PCB_OSCILLATOR:KC5032A_Foot_Print, symbol KC5032A
- removed U4: AD9833, Housings_SSOP:MSOP-10_3x3mm_Pitch0.5mm, symbol AD9833
- removed U6: LD1117S33TR_MIO, TO_SOT_Packages_SMD:SOT-223, symbol LD1117S33TR_MIO
- removed U?: ADG819, Housings_SSOP:MSOP-8_3x3mm_Pitch0.65mm, symbol ADG819
- removed U?: AD8421, symbol AD8421
- removed Y2: Crystal, Huellas:Crystal_SMD_XRCHA_Murata_Serie_W2,5mm_L2,0mm, symbol Crystal_Small
- added CLK?: KC5032A, Foot_Prints_PCB_OSCILLATOR:KC5032A_Foot_Print, symbol KC5032A
- added U?: LD1117S33TR_MIO, TO_SOT_Packages_SMD:SOT-223, symbol LD1117S33TR_MIO
- added U?: ADG819, Housings_SSOP:MSOP-8_3x3mm_Pitch0.65mm, symbol ADG819
- added U?: AD8421, Housings_SOIC:SOIC-8_3.9x4.9mm_Pitch1.27mm, symbol AD8421
- added U?: AD9833, Housings_SSOP:MSOP-10_3x3mm_Pitch0.5mm, symbol AD9833
- added Y?: XRCHA_16M, Huellas:Crystal_SMD_XRCHA_Murata_Serie_W2,5mm_L2,0mm, symbol XRCHA_16M
Connections:
- net BASE_WAVE: now also U?.8 (S2)
- net FSYNK_DDS_1: now also U?.8 (FSYNK)
- net GND: now also CLK?.2 (GND), U?.1 (GND), U?.2 (S1), U?.3 (GND), U?.4 (DGND), U?.9 (AGND)
- net MCLK_DDS_1: now also CLK?.3 (Output)
- net MODULATING_WAVE: now also U?.6 (IN)
- net SCLK_DDS_1: now also U?.7 (SCLK)
- net SDATA_DDS_1: now also U?.6 (SDATA)
- net VDD: now also CLK?.4 (Vcc), U?.2 (VDD), U?.4 (VDD)
- net XTAL1: now also Y?.1
- net XTAL2: now also Y?.2
- net at C32.2: now also U?.1 (COMP)
- net at C33.1, J14.2: now also U?.10 (VOUT)
- net at C25.1, C26.1: now also U?.3 (CAP)
- net at J10.1, J11.1: now also U?.5 (MCLK)
- net at J7.1, R21.2: now also CLK?.1 (_INH)
- net at C36.1, JP3.1: now also U?.2 (VO)
- net at C34.1, JP2.2: now also U?.3 (VI)
- net at J?.2: now also U?.1 (D)
Changed lines of the file:
@@
 LIBS:LIBERIA_PCB_OSCILLATOR
 LIBS:Resistencias_Proyecto
+LIBS:Sensado_Control_DC_5-cache
 LIBS:4_Wave_Generator-cache
 EELAYER 25 0
@@
 Comment4 ""
 $EndDescr
-$Comp
-L AD9833 U4
-U 1 1 59D306B1
-P 7990 5750
-F 0 "U4" H 7970 6020 60  0000 C CNN
-F 1 "AD9833" H 7960 5620 60  0000 C CNN
-F 2 "Housings_SSOP:MSOP-10_3x3mm_Pitch0.5mm" H 7790 5780 60  0001 C CNN
-F 3 "" H 7790 5780 60  0000 C CNN
-	1    7990 5750
-	1    0    0    -1
-$EndComp
 Text Label 7900 6620 1    60   ~ 0
 GND
@@
 $EndComp
 $Comp
-L LD1117S33TR_MIO U6
-U 1 1 59D306DB
-P 11050 1080
-F 0 "U6" H 11050 1180 50  0000 C CNN
-F 1 "LD1117S33TR_MIO" H 11050 1280 50  0000 C CNN
-F 2 "TO_SOT_Packages_SMD:SOT-223" H 11050 1180 50  0001 C CNN
-F 3 "" H 11050 1080 50  0001 C CNN
-	1    11050 1080
-	1    0    0    -1
-$EndComp
-$Comp
 L CONN_01X03 J1
 U 1 1 59D306DC
@@
 Wire Wire Line
 	12230 1030 12540 1030
-$Comp
-L Crystal_Small Y2
-U 1 1 59D306E7
-P 12270 2920
-F 0 "Y2" H 12270 3020 50  0000 C CNN
-F 1 "Crystal" H 12270 2820 50  0000 C CNN
-F 2 "Huellas:Crystal_SMD_XRCHA_Murata_Serie_W2,5mm_L2,0mm" H 12270 2920 50  0001 C CNN
-F 3 "" H 12270 2920 50  0001 C CNN
-	1    12270 2920
-	1    0    0    -1
-$EndComp
 $Comp
 L 20pF C21
@@
 $Comp
 L ADG819 U?
-U 1 1 59D73BBE
-P 14370 8010
-F 0 "U?" H 14230 8390 60  0000 C CNN
-F 1 "ADG819" H 14380 8010 60  0000 C CNN
-F 2 "Housings_SSOP:MSOP-8_3x3mm_Pitch0.65mm" H 14130 8290 60  0001 C CNN
-F 3 "" H 14370 8010 60  0000 C CNN
-	1    14370 8010
-	1    0    0    -1
-$EndComp
-$Comp
-L ADG819 U?
 U 1 1 59D744EC
 P 14390 5800
@@
 $EndComp
 $Comp
-L AD8421 U?
-U 1 1 59D78D88
-P 14530 3400
-F 0 "U?" H 14310 3710 60  0000 C CNN
-F 1 "AD8421" H 14520 3330 60  0000 C CNN
-F 2 "" H 14360 3100 60  0000 C CNN
-F 3 "" H 14360 3100 60  0000 C CNN
-	1    14530 3400
+L LD1117S33TR_MIO U?
+U 1 1 59D82649
+P 11050 1080
+F 0 "U?" H 11050 1330 50  0000 C CNN
+F 1 "LD1117S33TR_MIO" H 11050 1280 50  0000 C CNN
+F 2 "TO_SOT_Packages_SMD:SOT-223" H 11050 1180 50  0001 C CNN
+F 3 "" H 11050 1080 50  0001 C CNN
+	1    11050 1080
+	1    0    0    -1
+$EndComp
+$Comp
+L XRCHA_16M Y?
+U 1 1 59DAC6C5
+P 12270 2920
+F 0 "Y?" H 12270 3020 50  0000 C CNN
+F 1 "XRCHA_16M" H 12270 2820 50  0000 C CNN
+F 2 "Huellas:Crystal_SMD_XRCHA_Murata_Serie_W2,5mm_L2,0mm" H 12170 2920 50  0001 C CNN
+F 3 "" H 12270 2920 50  0000 C CNN
+	1    12270 2920
+	1    0    0    -1
+$EndComp
+$Comp
+L ADG819 U?
+U 1 1 59DB9A19
+P 14370 8010
+F 0 "U?" H 14230 8390 60  0000 C CNN
+F 1 "ADG819" H 14380 8010 60  0000 C CNN
+F 2 "Housings_SSOP:MSOP-8_3x3mm_Pitch0.65mm" H 14130 8290 60  0001 C CNN
+F 3 "" H 14370 8010 60  0000 C CNN
+	1    14370 8010
 	1    0    0    -1
 $EndComp
 $Comp
 L KC5032A CLK?
-U 1 1 59D7E65A
+U 1 1 59DD3EE5
 P 11220 5060
 F 0 "CLK?" H 11220 5260 60  0000 C CNN
@@
 	1    0    0    -1
 $EndComp
+$Comp
+L AD8421 U?
+U 1 1 59DEE87F
+P 14540 3400
+F 0 "U?" H 14320 3710 60  0000 C CNN
+F 1 "AD8421" H 14530 3330 60  0000 C CNN
+F 2 "Housings_SOIC:SOIC-8_3.9x4.9mm_Pitch1.27mm" H 14370 3100 60  0001 C CNN
+F 3 "" H 14370 3100 60  0000 C CNN
+	1    14540 3400
+	1    0    0    -1
+$EndComp
+$Comp
+L AD9833 U?
+U 1 1 59DF121D
+P 7990 5750
+F 0 "U?" H 7970 6020 60  0000 C CNN
+F 1 "AD9833" H 7960 5620 60  0000 C CNN
+F 2 "Housings_SSOP:MSOP-10_3x3mm_Pitch0.5mm" H 8140 4950 60  0001 C CNN
+F 3 "" H 7790 5780 60  0000 C CNN
+	1    7990 5750
+	1    0    0    -1
+$EndComp

Commit message: GENERADOR_V6
ESQUEMATICO LISTO PERO POR REVISAR
Parts:
- added P?: CON_MUX2, symbol CONN_01X02
Connections:
- net BASE_WAVE: now also J14.1; no longer U?.8 (S2)
- net MODULATED_WAVE_1: now also U?.6 (IN), P?.2 (P2)
- net MODULATING_WAVE: no longer U?.6 (IN)
- net WAVE_DDS_2: now also W?.1
- removed net WAVE_DDS_1: J14.1, W?.1
- new net MIN_SANGRADO: P?.1 (P1), U?.8 (S2)
Other:
- note added: "CONEXION DDEL SEGUNDO \nMUXTIPLEXOR"
- note added: "TO VARY GAIN\nOF AMPLIFIER"
- moved on the sheet: P4, P?, W?
