File: 4_Wave_Generador/4_Wave_Generator.sch (KiCad schematic (older format))
At the start: 117 parts, among them J1 RS232, J10 Jumper, J11 Jumper, J12 Jumper, J13 Jumper, J14 Jumper, J15 Jumper, J2 I2C, J4 RESET, J7 Jumper, P1 ECG INPUTS, P2 PIC_PROGRAMER, P3 SPI, P4 AD8232_CONTROL, P6 CONN_01X04, P7 CONN_01X04, P8 MCLK_EXTERNAL, SW1 SW_Push, SW2 RESET_PIC, Y1 Crystal_8MHz

Commit message: POWER_AMPLIFIER_FINISH
ULTIMOS CAMBIOS DE PLANOS EN PLACA DE MOSFET
Parts:
- removed C11, C8: 0.1uF, Capacitors_SMD:C_0805_HandSoldering, symbol 0.1uF
- removed C12, C9: 10uF, Capacitors_SMD:C_0805_HandSoldering, symbol 10uF
Other:
- moved on the sheet: C13, C14, C15, C16, C17
Changed lines of the file:
@@
 L 0.1uF C13
 U 1 1 59D306C5
-P 15210 1330
-F 0 "C13" H 15220 1400 50  0000 L CNN
-F 1 "0.1uF" H 15220 1250 50  0000 L CNN
-F 2 "Capacitors_SMD:C_0805_HandSoldering" H 15120 1300 50  0001 C CNN
-F 3 "" H 15220 1400 50  0001 C CNN
-F 4 "478-1395-2-ND" H 15320 1500 60  0001 C CNN "Digi-Key Part Number"
-	1    15210 1330
+P 14570 1360
+F 0 "C13" H 14580 1430 50  0000 L CNN
+F 1 "0.1uF" H 14580 1280 50  0000 L CNN
+F 2 "Capacitors_SMD:C_0805_HandSoldering" H 14480 1330 50  0001 C CNN
+F 3 "" H 14580 1430 50  0001 C CNN
+F 4 "478-1395-2-ND" H 14680 1530 60  0001 C CNN "Digi-Key Part Number"
+	1    14570 1360
 	1    0    0    -1
 $EndComp
@@
 L 10uF C15
 U 1 1 59D306C6
-P 15500 1330
-F 0 "C15" H 15510 1400 50  0000 L CNN
-F 1 "10uF" H 15510 1250 50  0000 L CNN
-F 2 "Capacitors_SMD:C_0805_HandSoldering" H 15410 1300 50  0001 C CNN
-F 3 "" H 15510 1400 50  0001 C CNN
-F 4 "490-5523-2-ND" H 15610 1500 60  0001 C CNN "25V"
-	1    15500 1330
-	1    0    0    -1
-$EndComp
-Text Label 15460 1590 2    60   ~ 0
-GND
-Text Label 15260 1060 0    60   ~ 0
+P 14860 1360
+F 0 "C15" H 14870 1430 50  0000 L CNN
+F 1 "10uF" H 14870 1280 50  0000 L CNN
+F 2 "Capacitors_SMD:C_0805_HandSoldering" H 14770 1330 50  0001 C CNN
+F 3 "" H 14870 1430 50  0001 C CNN
+F 4 "490-5523-2-ND" H 14970 1530 60  0001 C CNN "25V"
+	1    14860 1360
+	1    0    0    -1
+$EndComp
+Text Label 14820 1620 2    60   ~ 0
+GND
+Text Label 14620 1090 0    60   ~ 0
 VDD
 $Comp
@@
 	11160 10820 11480 10820
 Wire Wire Line
-	15210 1060 15500 1060
-Wire Wire Line
-	15500 1060 15500 1230
-Wire Wire Line
-	15500 1430 15500 1590
-Wire Wire Line
-	15500 1590 15210 1590
+	14570 1090 14860 1090
+Wire Wire Line
+	14860 1090 14860 1260
+Wire Wire Line
+	14860 1460 14860 1620
+Wire Wire Line
+	14860 1620 14570 1620
 Wire Notes Line
 	15810 4420 15810 2410
@@
 Text Notes 3770 9740 0    60   ~ 0
 DIGITAL BUSES AND CONNECTORS
-$Comp
-L 0.1uF C8
-U 1 1 59D306D8
-P 13100 1390
-F 0 "C8" H 13110 1460 50  0000 L CNN
-F 1 "0.1uF" H 13110 1310 50  0000 L CNN
-F 2 "Capacitors_SMD:C_0805_HandSoldering" H 13010 1360 50  0001 C CNN
-F 3 "" H 13110 1460 50  0001 C CNN
-F 4 "478-1395-2-ND" H 13210 1560 60  0001 C CNN "Digi-Key Part Number"
-	1    13100 1390
-	1    0    0    -1
-$EndComp
-$Comp
-L 10uF C9
-U 1 1 59D306D9
-P 13390 1390
-F 0 "C9" H 13400 1460 50  0000 L CNN
-F 1 "10uF" H 13400 1310 50  0000 L CNN
-F 2 "Capacitors_SMD:C_0805_HandSoldering" H 13300 1360 50  0001 C CNN
-F 3 "" H 13400 1460 50  0001 C CNN
-F 4 "490-5523-2-ND" H 13500 1560 60  0001 C CNN "25V"
-	1    13390 1390
-	1    0    0    -1
-$EndComp
-Text Label 13350 1650 2    60   ~ 0
-GND
-Text Label 13130 1120 0    60   ~ 0
-+12V
 Text Notes 9780 660  0    60   ~ 0
 Regulator
@@
 L 0.1uF C16
 U 1 1 59D306E2
-P 14640 1350
-F 0 "C16" H 14650 1420 50  0000 L CNN
-F 1 "0.1uF" H 14650 1270 50  0000 L CNN
-F 2 "Resistors_SMD:R_0805_HandSoldering" H 14550 1320 50  0001 C CNN
-F 3 "" H 14650 1420 50  0001 C CNN
-F 4 "478-1395-2-ND" H 14750 1520 60  0001 C CNN "Digi-Key Part Number"
-	1    14640 1350
+P 13670 1370
+F 0 "C16" H 13680 1440 50  0000 L CNN
+F 1 "0.1uF" H 13680 1290 50  0000 L CNN
+F 2 "Resistors_SMD:R_0805_HandSoldering" H 13580 1340 50  0001 C CNN
+F 3 "" H 13680 1440 50  0001 C CNN
+F 4 "478-1395-2-ND" H 13780 1540 60  0001 C CNN "Digi-Key Part Number"
+	1    13670 1370
 	1    0    0    -1
 $EndComp
@@
 L 0.1uF C17
 U 1 1 59D306E3
-P 14910 1350
-F 0 "C17" H 14920 1420 50  0000 L CNN
-F 1 "0.1uF" H 14920 1270 50  0000 L CNN
-F 2 "Resistors_SMD:R_0805_HandSoldering" H 14820 1320 50  0001 C CNN
-F 3 "" H 14920 1420 50  0001 C CNN
-F 4 "478-1395-2-ND" H 15020 1520 60  0001 C CNN "Digi-Key Part Number"
-	1    14910 1350
+P 13940 1370
+F 0 "C17" H 13950 1440 50  0000 L CNN
+F 1 "0.1uF" H 13950 1290 50  0000 L CNN
+F 2 "Resistors_SMD:R_0805_HandSoldering" H 13850 1340 50  0001 C CNN
+F 3 "" H 13950 1440 50  0001 C CNN
+F 4 "478-1395-2-ND" H 14050 1540 60  0001 C CNN "Digi-Key Part Number"
+	1    13940 1370
 	1    0    0    -1
 $EndComp
@@
 L 0.1uF C14
 U 1 1 59D306E4
-P 14360 1350
-F 0 "C14" H 14370 1420 50  0000 L CNN
-F 1 "0.1uF" H 14370 1270 50  0000 L CNN
-F 2 "Resistors_SMD:R_0805_HandSoldering" H 14270 1320 50  0001 C CNN
-F 3 "" H 14370 1420 50  0001 C CNN
-F 4 "478-1395-2-ND" H 14470 1520 60  0001 C CNN "Digi-Key Part Number"
-	1    14360 1350
+P 13390 1370
+F 0 "C14" H 13400 1440 50  0000 L CNN
+F 1 "0.1uF" H 13400 1290 50  0000 L CNN
+F 2 "Resistors_SMD:R_0805_HandSoldering" H 13300 1340 50  0001 C CNN
+F 3 "" H 13400 1440 50  0001 C CNN
+F 4 "478-1395-2-ND" H 13500 1540 60  0001 C CNN "Digi-Key Part Number"
+	1    13390 1370
 	1    0    0    -1
 $EndComp
@@
 Wire Wire Line
 	4350 10140 4350 10910
-Wire Wire Line
-	13100 1290 13100 1120
-Wire Wire Line
-	13100 1120 13390 1120
-Wire Wire Line
-	13390 1120 13390 1290
-Wire Wire Line
-	13390 1490 13390 1650
-Wire Wire Line
-	13390 1650 13100 1650
-Wire Wire Line
-	13100 1650 13100 1490
 Wire Notes Line
 	9700 550  9700 1620
@@
 Connection ~ 11050 1510
 Wire Wire Line
-	14910 1250 14910 1200
-Wire Wire Line
-	14910 1200 14360 1200
-Wire Wire Line
-	14360 1200 14360 1250
-Wire Wire Line
-	14640 1250 14640 1200
-Connection ~ 14640 1200
-Wire Wire Line
-	14910 1450 14910 1540
-Wire Wire Line
-	14910 1540 14360 1540
-Wire Wire Line
-	14360 1540 14360 1450
-Wire Wire Line
-	14640 1450 14640 1540
-Connection ~ 14640 1540
-Text Label 14470 1200 0    60   ~ 0
+	13940 1270 13940 1220
+Wire Wire Line
+	13940 1220 13390 1220
+Wire Wire Line
+	13390 1220 13390 1270
+Wire Wire Line
+	13670 1270 13670 1220
+Connection ~ 13670 1220
+Wire Wire Line
+	13940 1470 13940 1560
+Wire Wire Line
+	13940 1560 13390 1560
+Wire Wire Line
+	13390 1560 13390 1470
+Wire Wire Line
+	13670 1470 13670 1560
+Connection ~ 13670 1560
+Text Label 13500 1220 0    60   ~ 0
 VDD
-Text Label 14440 1540 0    60   ~ 0
+Text Label 13470 1560 0    60   ~ 0
 GND
 $Comp
@@
 Text Notes 11210 2910 0    60   ~ 0
 CRYSTAL \nOSCILLATOR
-$Comp
-L 0.1uF C11
-U 1 1 59D306F0
-P 13720 1390
-F 0 "C11" H 13730 1460 50  0000 L CNN
-F 1 "0.1uF" H 13730 1310 50  0000 L CNN
-F 2 "Capacitors_SMD:C_0805_HandSoldering" H 13630 1360 50  0001 C CNN
-F 3 "" H 13730 1460 50  0001 C CNN
-F 4 "478-1395-2-ND" H 13830 1560 60  0001 C CNN "Digi-Key Part Number"
-	1    13720 1390
-	1    0    0    -1
-$EndComp
-$Comp
-L 10uF C12
-U 1 1 59D306F1
-P 14010 1390
-F 0 "C12" H 14020 1460 50  0000 L CNN
-F 1 "10uF" H 14020 1310 50  0000 L CNN
-F 2 "Capacitors_SMD:C_0805_HandSoldering" H 13920 1360 50  0001 C CNN
-F 3 "" H 14020 1460 50  0001 C CNN
-F 4 "490-5523-2-ND" H 14120 1560 60  0001 C CNN "25V"
-	1    14010 1390
-	1    0    0    -1
-$EndComp
-Text Label 13970 1650 2    60   ~ 0
-GND
-Text Label 13750 1120 0    60   ~ 0
-+5V
-Wire Wire Line
-	13720 1290 13720 1120
-Wire Wire Line
-	13720 1120 14010 1120
-Wire Wire Line
-	14010 1120 14010 1290
-Wire Wire Line
-	14010 1490 14010 1650
-Wire Wire Line
-	14010 1650 13720 1650
-Wire Wire Line
-	13720 1650 13720 1490
 Text Notes 13050 1000 0    60   ~ 0
 DECUPLING CAPACITORS
@@
 $EndComp
 Wire Wire Line
-	15210 1590 15210 1430
-Wire Wire Line
-	15210 1230 15210 1060
+	14570 1620 14570 1460
+Wire Wire Line
+	14570 1260 14570 1090
 Wire Notes Line
 	15840 890  15840 1750

Commit message: GENERADOR V_7
TOCAS LAS CONEXIONES
Parts:
- removed P?: SALIDAS_DIG_ATMEGA, symbol CONN_01X11
- removed P?: SALIDAS_DIG_PIC, symbol CONN_01X05
- added P10: INPUT_ADC_PIC, symbol CONN_01X02
- added P11: PWM_MUX1, symbol CONN_01X02
- added P14: OUTPUT_TARJET, symbol CONN_01X02
- added P15: OUTPUT_DIG_PIC, symbol CONN_01X04
- added P16: OUTPUT_DIG_ATMEGA328P, symbol CONN_01X12
- added P9: SPI_AD9833, symbol CONN_01X03
- added R18, R19: 10K, Resistors_SMD:R_0805_HandSoldering, symbol 10K
- gave numbers to parts that had none: 30
Connections:
- net +vs is gone; now on net VDD: C7.2, R12.1, U2.17 (+VS)
- net +12V: now also U8.8 (+Vs)
- net -12V: now also U8.5 (-Vs)
- net ADC_1: now also P10.1 (P1)
- net ADC_2: now also P10.2 (P2)
- net A_AD5270_1: now also U8.2 (Rg)
- net BASE_WAVE: no longer J13.1
- net FSYNK_DDS_1: now also P9.3 (P3)
- net GND: now also P13.2 (P2), U2.21 (GND), U8.1 (-IN), P11.2 (P2), P14.2 (P2), P15.1 (P1), R18.1, R19.1; no longer U6.2 (S1), U7.2 (S1)
- net MIN_SANGRADO: now also U6.6 (IN); no longer U6.8 (S2)
- net MODULATED_WAVE_1: now also U6.8 (S2); no longer P13.2 (P2), U6.6 (IN)
- net MODULATED_WAVE_2: now also U8.4 (+IN)
- net MODULATING_WAVE: now also P11.1 (P1)
- net PB0: now also P16.2 (P2)
- net PB1: now also P16.1 (P1)
- net PC0: now also P16.9 (P9)
- net PC1: now also P16.8 (P8)
- net PC2: now also P16.7 (P7)
- net PC3: now also P16.6 (P6)
- net PD2: now also P16.10 (P10)
- net PD3: now also P16.11 (P11)
- net PD4: now also P16.12 (P12)
- net PD5: now also P16.5 (P5)
- net PD6: now also P16.4 (P4)
- net PD7: now also P16.3 (P3)
- net RC1_PIC: now also P15.2 (P2)
- net RC2_PIC: now also P15.3 (P3)
- net RC3_PIC: now also P15.4 (P4)
- net SCLK_DDS_1: now also P9.2 (P2)
- net SDATA_DDS_1: now also P9.1 (P1)
- net W_AD5270_1: now also U8.3 (Rg)
- net at J13.2: now also U8.7 (Vout)
- net at J12.1: now also U8.6 (REF)
- net WAVE_DDS_2 renamed VOUT_AMPLIFIER
- net VOUT_AMPLIFIER: now also J13.1, P14.1 (P1)
- new net MUX_1_S1: R19.2, U7.2 (S1)
- new net MUX_2_S1: R18.2, U6.2 (S1)
Other:
- note added: "ADC DEL PIC\n"
- note added: "LOGIC CONTROL INPUT\n"
- note added: "MUX_1\n"
- note added: "MUX_2"
- note added: "OUTPUT GAVE GENERATOR"
- note removed: "CONEXION DDEL SEGUNDO \nMUXTIPLEXOR"
- moved on the sheet: C33, J1, J14, J2, J3, J4, P13, P2, P3
