File: 4_Wave_Generador/4_Wave_Generator.kicad_pcb (KiCad board)
At the start: 2 copper layers, 100 x 100 mm, 134 parts, among them J10 Jumper, J11 Jumper, J12 Jumper, J13 Jumper, J14 Jumper, J15 Jumper, J4 RESET, J5 Jumper, J6 Jumper, J7 Jumper, J8 Jumper, P1 ECG INPUTS, P10 INPUT_ADC_PIC, P11 DIG_ATMEGA, P12 RG_8421, P13 OUTPUT_DIG_PIC, P14 OUTPUT_TARJET, P15 MUX_S1, P16 DIG_MICRO, P17 SUPPLY_-12V, P18 RS232, P19 I2C, P2 PIC_PROGRAMER, P20 DIG_ATMEGA2, P3 SPI_MICRO, P31 TORNILLO, P32 TORNILLO, P33 TORNILLO, P34 TORNILLO, P35 RS232_PIC, P4 AD8232_CONTROL, P5 OXIMETRO, P6 SUPPLY_12V, P7 SUPPLY_VDD, SW1 SW_Push, SW2 RESET_PIC, U1 PIC16F688, U3 ATMEGA328P-AU_MIO, U4 AD9833, U5 LD1117S33TR_MIO, Y1 Crystal_8MHz, Y2 XRCHA_16M

Commit message: ULTIMO DISEÑO
FIN PCBS
Parts:
- moved G*** 5.56 mm to (87.6, 106.7)
Routing:
- net /VDD: track 591.8 -> 586.6 mm, vias 30 -> 27
Changed lines of the file:
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@@
     (thickness 1.6)
     (drawings 9)
-    (tracks 1875)
+    (tracks 1866)
     (zones 0)
     (modules 134)
@@
     (tags "capacitor 0805")
     (attr smd)
-    (fp_text reference C26 (at -0.74 -1.57 180) (layer F.SilkS)
+    (fp_text reference C26 (at 2.514 -1.564 180) (layer F.SilkS)
       (effects (font (size 1 1) (thickness 0.15)))
     )
@@
     (descr "Through hole straight pin header, 1x02, 2.54mm pitch, single row")
     (tags "Through hole pin header THT 1x02 2.54mm single row")
-    (fp_text reference J10 (at 0 -2.33 270) (layer F.SilkS)
+    (fp_text reference J10 (at 3.408 0.814 270) (layer F.SilkS)
       (effects (font (size 1 1) (thickness 0.15)))
     )
@@
   (module Huellas:AD8232_ECG (layer F.Cu)
     (at 97.15 118.9)
-    (fp_text reference AD8232 (at 1.656 3.274) (layer F.SilkS)
+    (fp_text reference AD8232 (at 1.656 4.29) (layer F.SilkS)
       (effects (font (size 1 1) (thickness 0.15)))
     )
@@
   )
   (module Logos_Fuentes:UIS (layer F.Cu)
-    (at 84.32 111.15)
+    (at 87.63 106.68)
     (fp_text reference G*** (at 0 0) (layer F.SilkS) hide
       (effects (font (thickness 0.3)))
@@
   (segment (start 153.45 65.8) (end 153.45 66.2) (width 2) (layer F.Cu) (net 11))
   (segment (start 98.298 81.534) (end 98.298 81.442) (width 2) (layer B.Cu) (net 11))
-  (via (at 100.11 79.63) (size 0.6) (drill 0.4) (layers F.Cu B.Cu) (net 11))
   (segment (start 98.298 81.442) (end 100.11 79.63) (width 2) (layer B.Cu) (net 11))
-  (segment (start 100.11 79.63) (end 100.156 79.676) (width 2) (layer F.Cu) (net 11))
-  (segment (start 100.156 79.676) (end 100.11 79.63) (width 2) (layer F.Cu) (net 11))
-  (segment (start 100.11 79.63) (end 100.11 79.722) (width 2) (layer F.Cu) (net 11))
-  (segment (start 98.298 81.534) (end 98.298 81.552) (width 2) (layer F.Cu) (net 11))
-  (segment (start 98.298 81.552) (end 96.62 83.23) (width 2) (layer F.Cu) (net 11))
-  (via (at 96.62 83.23) (size 0.6) (drill 0.4) (layers F.Cu B.Cu) (net 11))
   (segment (start 96.62 83.23) (end 96.611 83.221) (width 2) (layer B.Cu) (net 11))
   (segment (start 96.611 83.221) (end 96.62 83.23) (width 2) (layer B.Cu) (net 11))
@@
   (segment (start 121.412 90.932) (end 120.396 90.932) (width 0.4) (layer F.Cu) (net 11))
   (segment (start 122.025 91.545) (end 121.412 90.932) (width 0.4) (layer F.Cu) (net 11))
-  (segment (start 100.11 79.722) (end 98.298 81.534) (width 2) (layer F.Cu) (net 11))
   (segment (start 89.408 104.394) (end 90.424 104.394) (width 2) (layer F.Cu) (net 11))
   (segment (start 90.424 104.394) (end 96.266 104.394) (width 2) (layer F.Cu) (net 11))
@@
   (segment (start 98.298 81.534) (end 96.62 83.212) (width 2) (layer B.Cu) (net 11))
   (segment (start 96.62 83.212) (end 91.694 88.138) (width 2) (layer B.Cu) (net 11))
-  (via (at 98.298 81.534) (size 0.6) (drill 0.4) (layers F.Cu B.Cu) (net 11))
   (segment (start 107.696 104.394) (end 111.506 104.394) (width 2) (layer F.Cu) (net 11))
   (segment (start 111.506 104.394) (end 118.11 104.394) (width 2) (layer F.Cu) (net 11))
@@
   )
   (zone (net 9) (net_name /GND) (layer F.Cu) (hatch edge 0.508)
-    (connect_pads yes (clearance 0.508))
+    (connect_pads (clearance 0.508))
     (min_thickness 0.254)
     (fill yes (arc_segments 16) (thermal_gap 0.508) (thermal_bridge_width 0.508))
@@
   )
   (zone (net 10) (net_name /+12V) (layer F.Cu) (hatch edge 0.508)
-    (connect_pads yes (clearance 0.508))
+    (connect_pads (clearance 0.508))
     (min_thickness 0.254)
     (fill yes (arc_segments 16) (thermal_gap 0.508) (thermal_bridge_width 0.508))
@@
   )
   (zone (net 11) (net_name /VDD) (layer F.Cu) (hatch edge 0.508)
-    (connect_pads yes (clearance 0.508))
+    (connect_pads (clearance 0.508))
     (min_thickness 0.254)
     (fill yes (arc_segments 16) (thermal_gap 0.508) (thermal_bridge_width 0.508))
@@
   )
   (zone (net 11) (net_name /VDD) (layer F.Cu) (hatch edge 0.508)
-    (connect_pads yes (clearance 0.508))
+    (connect_pads (clearance 0.508))
     (min_thickness 0.254)
     (fill yes (arc_segments 16) (thermal_gap 0.508) (thermal_bridge_width 0.508))
@@
   )
   (zone (net 21) (net_name "Net-(C36-Pad1)") (layer F.Cu) (hatch edge 0.508)
-    (connect_pads yes (clearance 0.508))
+    (connect_pads (clearance 0.508))
     (min_thickness 0.254)
     (fill yes (arc_segments 16) (thermal_gap 0.508) (thermal_bridge_width 0.508))
@@
   )
   (zone (net 20) (net_name "Net-(C34-Pad1)") (layer F.Cu) (hatch edge 0.508)
-    (connect_pads yes (clearance 0.508))
+    (connect_pads (clearance 0.508))
     (min_thickness 0.254)
     (fill yes (arc_segments 16) (thermal_gap 0.508) (thermal_bridge_width 0.508))
