File: 3_Power_Amplifier/3_Power_Amplifier/3_Power_Amplifier.kicad_pcb (KiCad board)
At the start: 2 copper layers, 100 x 100 mm, 24 parts, among them P1 SIGNAL_INPUT_SMA, P10 SWITCHED_POWER_INV, P11 SIGNAL_INPUT, P12 SWITCHED_POWER_INV, P2 SWITCHED_POWER_INV, P3 ISLETA, P4 ISLETA, P5 ISLETA, P6 ISLETA, P7 SIGNAL_INPUT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

Commit message: GENERADOR_V8
ORGANIZACION DE ELEMENTOS
Parts:
- removed R1, R3, R5, R7: 100, libreria_Power_Amplifier_huellas:INV_R_0805_HandSoldering
- removed R2, R4, R6, R8: 10K, libreria_Power_Amplifier_huellas:INV_R_0805_HandSoldering
- added 100: 100, Resistors_SMD:R_0805_HandSoldering, B.Cu at (104.0, 105.1)
- added 100: 100, Resistors_SMD:R_0805_HandSoldering, B.Cu at (123.1, 105.3)
- added 100: 100, Resistors_SMD:R_0805_HandSoldering, B.Cu at (141.7, 104.8)
- added 100: 100, Resistors_SMD:R_0805_HandSoldering, B.Cu at (160.7, 105.3)
- added 10K: 10K, Resistors_SMD:R_0805_HandSoldering, B.Cu at (107.8, 105.2)
- added 10K: 10K, Resistors_SMD:R_0805_HandSoldering, B.Cu at (127.0, 105.2)
- added 10K: 10K, Resistors_SMD:R_0805_HandSoldering, B.Cu at (145.6, 104.8)
- added 10K: 10K, Resistors_SMD:R_0805_HandSoldering, B.Cu at (164.7, 105.2)
Routing:
- net (no net): track 18.5 -> 0.00 mm
- net /DDS: track 171.8 -> 184.5 mm, vias 14 -> 12
- net /GND: track 948.5 -> 952.7 mm, vias 210 -> 232
Other:
- net class vias added: clearance 0.2, trace_width 0.6, via_dia 0.6, via_drill 0.4

Commit message: GENERADOR V_14
ULTIMO DISEÑO CON LOGOS
Parts:
- added G***: LOGO, Logos_Fuentes:SBS_22mm, B.Cu at (151.9, 81.3)
- added G***: LOGO, Logos_Fuentes:CMOS, B.Cu at (157.2, 53.6)
- added G***: LOGO, Logos_Fuentes:Colombia, B.Cu at (143.0, 53.8)
- added G***: LOGO, Logos_Fuentes:UIS, B.Cu at (106.2, 53.8)
Other:
- board text added: "3 POWER AMPLIFIER _ 1"
- board text added: "Colombia"
- board text removed: "3_POWER AMPLIFIER PART_1"

Commit message: ULTIMO DISEÑO
FIN PCBS
Parts:
- removed 100 (x4): 100, Resistors_SMD:R_0805_HandSoldering
- removed 10K (x4): 10K, Resistors_SMD:R_0805_HandSoldering
- added R1: 100, Resistors_SMD:R_0805_HandSoldering, B.Cu at (104.1, 105.2)
- added R2: 10K, Resistors_SMD:R_0805_HandSoldering, B.Cu at (108.0, 105.2)
- added R3: 100, Resistors_SMD:R_0805_HandSoldering, B.Cu at (122.9, 105.2)
- added R4: 10K, Resistors_SMD:R_0805_HandSoldering, B.Cu at (127.0, 105.2)
- added R5: 100, Resistors_SMD:R_0805_HandSoldering, B.Cu at (141.7, 105.2)
- added R6: 10K, Resistors_SMD:R_0805_HandSoldering, B.Cu at (145.5, 105.2)
- added R7: 100, Resistors_SMD:R_0805_HandSoldering, B.Cu at (160.8, 105.2)
- added R8: 10K, Resistors_SMD:R_0805_HandSoldering, B.Cu at (164.6, 105.2)
- Q1, Q2, Q3, Q4: footprint libreria_Power_Amplifier_huellas:TO-220_Ver_Disipador -> libreria_Power_Amplifier_huellas:NUEVO_TO-220_Ver_Disipador
- moved G*** 6.65 mm to (112.8, 53.1)
- moved G*** 2.34 mm to (144.8, 52.3)
- moved G*** 1.48 mm to (158.5, 52.8)
- moved G*** 0.57 mm to (151.6, 81.8)
Other:
- board text added: "003 POWER AMPLIFIER _ 1"
- board text removed: "3 POWER AMPLIFIER _ 1"
